Commit message: Bugok kijavítva: villogó pálya és kamerakép alsó része nem látszódik

File: race_car_description/urdf/camera.xacro (robot description, xacro)
@@ -59,5 +59,5 @@
 			<sensor type="camera" name="camera1">
 				<update_rate>30.0</update_rate>
-				<visualize>true</visualize>
+				<visualize>false</visualize>
 				<camera name="head">
 					<!-- FOV: 80 degrees -->
@@ -69,7 +69,7 @@
 					</image>
 					<clip>
-						<!-- <near>0.02</near>
-						<far>300</far> -->
-						<near>0.1</near>
+						<near>0.02</near>
+						<!-- <far>300</far> -->
+						<!-- <near>0.1</near> -->
 						<far>25</far>
 					</clip>

File: race_car_description/urdf/f1_car.xacro (robot description, xacro)
@@ -35,32 +35,33 @@
   <xacro:property name="deg_to_rad" value="0.01745329251994329577"/>
   <xacro:property name="mass_multiplier" value="10"/>
+  <xacro:property name="scale" value="32"/>
   <!-- Robot base dimensions -->
-  <xacro:property name="base_length" value="${5.5 / 32}" />
-  <xacro:property name="base_width" value="${2.0 / 32}" />
-  <xacro:property name="base_height" value="${1.0 / 32}" />
-  <xacro:property name="base_mass" value="${0.025 * mass_multiplier}" />
+  <xacro:property name="base_length" value="${5.5 / scale}" />
+  <xacro:property name="base_width" value="${2.0 / scale}" />
+  <xacro:property name="base_height" value="${1.0 / scale}" />
+  <xacro:property name="base_mass" value="${850 / (scale*scale*scale) * mass_multiplier}" />
   <!-- Wheel link dimensions -->
-  <xacro:property name="wheel_radius" value="${18*0.0254/2 / 32}" />
-  <xacro:property name="wheel_thickness" value="${0.35 / 32}" />
-  <xacro:property name="wheel_mass" value="${0.00032 * mass_multiplier}" />
+  <xacro:property name="wheel_radius" value="${18*0.0254/2 / scale}" />
+  <xacro:property name="wheel_thickness" value="${0.35 / scale}" />
+  <xacro:property name="wheel_mass" value="${10.5 / (scale*scale*scale) * mass_multiplier}" />
   <!-- Steering link dimensions -->
   <xacro:property name="steer_radius" value="${wheel_radius / 2}" />
   <xacro:property name="steer_thickness" value="${wheel_thickness / 4}" />
-  <xacro:property name="steer_mass" value="${0.00032 * mass_multiplier}" />
+  <xacro:property name="steer_mass" value="${10.5 / (scale*scale*scale) * mass_multiplier}" />
   <!-- Axle positions -->
-  <xacro:property name="wheelbase" value="${3.6 / 32}" />
-  <xacro:property name="ride_height" value="${0.032 / 32}" />
-  <xacro:property name="axle_offset_rear" value="0" />
-  <!-- <xacro:property name="axle_offset_rear" value="${wheel_radius}" /> -->
+  <xacro:property name="wheelbase" value="${3.6 / scale}" />
+  <xacro:property name="ride_height" value="${0.032 / scale}" />
+  <!-- <xacro:property name="axle_offset_rear" value="0" /> -->
+  <xacro:property name="axle_offset_rear" value="${wheel_radius}" />
   <xacro:property name="axle_offset_front" value="${base_length - axle_offset_rear - wheelbase}" />
   <xacro:property name="axle_height" value="${-base_height/2 - ride_height + wheel_radius}" />
   <xacro:property name="steer_offset" value="${steer_thickness}" />
   <!-- Camera dimensions -->
-	<xacro:property name="camera_size" value="${0.2 / 32}"/>
+	<xacro:property name="camera_size" value="${0.2 / scale}"/>
 	<xacro:property name="camera_width" value="${camera_size}"/>
 	<xacro:property name="camera_thickness" value="${camera_size/2}"/>
 	<xacro:property name="camera_height" value="${camera_size*2/3}"/>
-	<xacro:property name="camera_mass" value="${0.00003 * mass_multiplier}"/>
-	<xacro:property name="camera_forward_tilt_deg" value="0"/>
+	<xacro:property name="camera_mass" value="${1 / (scale*scale*scale) * mass_multiplier}"/>
+	<xacro:property name="camera_forward_tilt_deg" value="10"/>
   <!-- Base link -->
   <link name="base_link">

Commit message: Vizuális modell implementálása

File: race_car_description/urdf/camera.xacro (robot description, xacro)
@@ -69,5 +69,5 @@
 					</image>
 					<clip>
-						<near>0.02</near>
+						<near>0.01</near>
 						<!-- <far>300</far> -->
 						<!-- <near>0.1</near> -->

File: race_car_description/urdf/f1_car.xacro (robot description, xacro)
@@ -53,5 +53,6 @@
   <xacro:property name="ride_height" value="${0.032 / scale}" />
   <!-- <xacro:property name="axle_offset_rear" value="0" /> -->
-  <xacro:property name="axle_offset_rear" value="${wheel_radius}" />
+  <!-- <xacro:property name="axle_offset_rear" value="${wheel_radius}" /> -->
+  <xacro:property name="axle_offset_rear" value="${1.050 / scale}" />
   <xacro:property name="axle_offset_front" value="${base_length - axle_offset_rear - wheelbase}" />
   <xacro:property name="axle_height" value="${-base_height/2 - ride_height + wheel_radius}" />
@@ -63,5 +64,12 @@
 	<xacro:property name="camera_height" value="${camera_size*2/3}"/>
 	<xacro:property name="camera_mass" value="${1 / (scale*scale*scale) * mass_multiplier}"/>
-	<xacro:property name="camera_forward_tilt_deg" value="10"/>
+	<xacro:property name="camera_forward_tilt_deg" value="0"/>
+	<!-- <xacro:property name="camera_x" value="${base_length/2+camera_thickness/2}"/> -->
+	<xacro:property name="camera_y" value="0"/>
+	<!-- <xacro:property name="camera_z" value="${base_height/2-camera_height/2}"/> -->
+	<!-- <xacro:property name="camera_x" value="${-1.41 / scale + camera_thickness/2}"/>
+	<xacro:property name="camera_z" value="${0.82 / scale - camera_height/2}"/> -->
+	<xacro:property name="camera_x" value="${2.75 / scale + camera_thickness/2}"/>
+	<xacro:property name="camera_z" value="${-0.192 / scale - camera_height/2}"/>
   <!-- Base link -->
   <link name="base_link">
@@ -69,7 +77,8 @@
       <origin xyz="0 0 0" rpy="0 0 0"/>
       <geometry>
-        <box size="${base_length} ${base_width} ${base_height}"/>
+        <!-- <box size="${base_length} ${base_width} ${base_height}"/> -->
+        <mesh filename="package://race_car_gazebo/meshes/f1_car_body.dae"/>
       </geometry>
-      <material name="green" />
+      <!-- <material name="green" /> -->
     </visual>
     <collision>
@@ -84,4 +93,8 @@
         x="${base_length}" y="${base_width}" z="${base_height}" />
   </link>
+  <!-- Colour -->
+  <!-- <gazebo reference="base_link">
+    <material>Gazebo/Green</material>
+  </gazebo> -->
   <!-- Camera -->
   <xacro:camera
@@ -91,5 +104,5 @@
     camera_height="${camera_height}"
     forward_tilt="${camera_forward_tilt_deg}">
-    <origin xyz="${base_length/2+camera_thickness/2} 0 ${base_height/2-camera_height/2}"
+    <origin xyz="${camera_x} ${camera_y} ${camera_z}"
             rpy="0 ${camera_forward_tilt_deg * deg_to_rad} 0"/>
   </xacro:camera>
@@ -152,22 +165,30 @@
     name="rear_right"
     parent="base"
+    reflect="-1"
     wheel_radius="${wheel_radius}"
     wheel_thickness="${wheel_thickness}"
-    wheel_mass="${wheel_mass}">
-    <origin xyz="${-base_length/2+axle_offset_rear} ${-base_width/2-wheel_thickness/2} ${axle_height}"
-            rpy="${-90 * deg_to_rad} 0 0"/>
+    wheel_mass="${wheel_mass}"
+    base_length="${base_length}"
+    base_width="${base_width}"
+    axle_offset="${axle_offset_rear}"
+    axle_height="${axle_height}">
+    <!-- <origin xyz="${-base_length/2+axle_offset_rear} ${-base_width/2-wheel_thickness/2} ${axle_height}"  -->
+    <!-- <origin xyz="${-base_length/2+axle_offset_rear} ${-base_width/2+wheel_thickness/2} ${axle_height}"
+            rpy="${-90 * deg_to_rad} 0 0"/> -->
   </xacro:rear_wheel_lr>
   <xacro:rear_wheel_lr
     name="rear_left"
     parent="base"
+    reflect="1"
     wheel_radius="${wheel_radius}"
     wheel_thickness="${wheel_thickness}"
-    wheel_mass="${wheel_mass}">
-    <origin xyz="${-base_length/2+axle_offset_rear} ${+base_width/2+wheel_thickness/2} ${axle_height}"
-            rpy="${-90 * deg_to_rad} 0 0"/>
+    wheel_mass="${wheel_mass}"
+    base_length="${base_length}"
+    base_width="${base_width}"
+    axle_offset="${axle_offset_rear}"
+    axle_height="${axle_height}">
+    <!-- <origin xyz="${-base_length/2+axle_offset_rear} ${+base_width/2+wheel_thickness/2} ${axle_height}"  -->
+    <!-- <origin xyz="${-base_length/2+axle_offset_rear} ${+base_width/2-wheel_thickness/2} ${axle_height}"
+            rpy="${-90 * deg_to_rad} 0 0"/> -->
   </xacro:rear_wheel_lr>
-  <!-- Colour -->
-  <gazebo reference="base_link">
-    <material>Gazebo/Green</material>
-  </gazebo>
 </robot>

File: race_car_description/urdf/wheel.xacro (robot description, xacro)
@@ -15,5 +15,5 @@
   <xacro:property name="steer_effort" value="10.0"/>
   <xacro:property name="steer_velocity" value="5.0"/>
-  <xacro:property name="steer_limit_deg" value="45.0"/>
+  <xacro:property name="steer_limit_deg" value="30.0"/>
   <!-- Bicycle model front steering link (required for steer_drive_controller) -->
   <xacro:macro name="front_steer"
@@ -29,5 +29,5 @@
       steer_height">
     <link name="${name}_steer_link">
-      <visual>
+      <!-- <visual>
         <origin xyz="0 0 0" rpy="0 0 0"/>
         <geometry>
@@ -35,5 +35,5 @@
         </geometry>
         <material name="yellow" />
-      </visual>
+      </visual> -->
       <collision>
         <origin xyz="0 0 0" rpy="0 0 0"/>
@@ -53,6 +53,7 @@
       <axis xyz="0 0 1"/>
       <limit effort="${steer_effort}"
-             lower="${-180.0 * deg_to_rad}" upper="${180.0 * deg_to_rad}"
+             lower="${steer_limit_deg * deg_to_rad * -1.0}" upper="${steer_limit_deg * deg_to_rad}"
              velocity="${steer_velocity}"/>
+             <!-- lower="${-180.0 * deg_to_rad}" upper="${180.0 * deg_to_rad}" -->
     </joint>
     <!-- <transmission name="${name}_steer_joint_trans">
@@ -66,7 +67,7 @@
       </joint>
     </transmission> -->
-    <gazebo reference="${name}_steer_link">
+    <!-- <gazebo reference="${name}_steer_link">
       <material>Gazebo/Yellow</material>
-    </gazebo>
+    </gazebo> -->
   </xacro:macro>
   <!-- Car steering model front (steerable) wheel links (left/right) -->
@@ -88,12 +89,11 @@
       axle_height">
     <link name="${name}_steer_link">
-      <visual>
+      <!-- <visual>
         <origin xyz="0 0 0" rpy="0 0 0"/>
         <geometry>
           <cylinder radius="${steer_radius}" length="${steer_thickness}"/>
-					<!-- <mesh filename="package://robotrendszerek_projekt/meshes/f1_car_wheel.dae"/> -->
         </geometry>
         <material name="blue" />
-      </visual>
+      </visual> -->
       <collision>
         <origin xyz="0 0 0" rpy="0 0 0"/>
@@ -110,5 +110,6 @@
       <parent link="${parent}_link"/>
       <child link="${name}_steer_link"/>
-      <origin xyz="${base_length/2-axle_offset} ${reflect*(base_width/2+wheel_thickness/2)} ${steer_height}" rpy="0 0 0"/>
+      <!-- <origin xyz="${base_length/2-axle_offset} ${reflect*(base_width/2+wheel_thickness/2)} ${steer_height}" rpy="0 0 0"/> -->
+      <origin xyz="${base_length/2-axle_offset} ${reflect*(base_width/2-wheel_thickness/2)} ${steer_height}" rpy="0 0 0"/>
       <axis xyz="0 0 1"/>
       <limit effort="${steer_effort}"
@@ -118,7 +119,8 @@
     <link name="${name}_wheel_link">
       <visual>
-        <origin xyz="0 0 0" rpy="0 0 0"/>
-        <geometry>
-          <cylinder radius="${wheel_radius}" length="${wheel_thickness}"/>
+        <origin xyz="0 0 0" rpy="${(1-reflect)/2 * 180 * deg_to_rad} 0 0"/>
+        <geometry>
+          <!-- <cylinder radius="${wheel_radius}" length="${wheel_thickness}"/> -->
+          <mesh filename="package://race_car_gazebo/meshes/f1_car_wheel_front.dae"/>
         </geometry>
         <material name="red" />
@@ -161,13 +163,13 @@
       </joint>
     </transmission> -->
-    <gazebo reference="${name}_steer_link">
+    <!-- <gazebo reference="${name}_steer_link">
       <material>Gazebo/Blue</material>
-    </gazebo>
+    </gazebo> -->
     <gazebo reference="${name}_wheel_link">
-      <material>Gazebo/Red</material>
+      <!-- <material>Gazebo/Red</material> -->
       <mu1 value="1.0"/>
 			<mu2 value="1.0"/>
-			<kp value="10000000.0" />
-			<kd value="1.0" />
+			<kp value="100000.0" />
+			<kd value="10.0" />
 			<fdir1 value="1 0 0"/>
     </gazebo>
@@ -175,4 +177,52 @@
   <!-- Bicycle model rear wheel link (required for steer_drive_controller) -->
   <xacro:macro name="rear_wheel"
+    params="
+      name
+      parent
+      wheel_radius
+      wheel_thickness
+      wheel_mass
+      *origin">
+    <link name="${name}_wheel_link">
+      <!-- <visual>
+        <origin xyz="0 0 0" rpy="0 0 0"/>
+        <geometry>
+          <cylinder radius="${wheel_radius}" length="${wheel_thickness}"/>
+        </geometry>
+        <material name="yellow" />
+      </visual> -->
+      <collision>
+        <origin xyz="0 0 0" rpy="0 0 0"/>
+        <geometry>
+          <cylinder radius="${wheel_radius}" length="${wheel_thickness}"/>
+        </geometry>
+      </collision>
+      <xacro:solid_cylinder_inertial
+          rpy="0 0 0" xyz="0 0 0"
+          mass="${wheel_mass}"
+          radius="${wheel_radius}" length="${wheel_thickness}" />
+    </link>
+    <joint name="${name}_wheel_joint" type="continuous">
+      <parent link="${parent}_link"/>
+      <child link="${name}_wheel_link"/>
+      <xacro:insert_block name="origin"/>
+      <axis xyz="0 0 1"/>
+    </joint>
+    <!-- <transmission name="${name}_wheel_joint_trans">
+      <type>transmission_interface/SimpleTransmission</type>
+      <actuator name="${name}_wheel_joint_motor">
+        <mechanicalReduction>1</mechanicalReduction>
+        <hardwareInterface>hardware_interface/VelocityJointInterface</hardwareInterface>
+      </actuator>
+      <joint name="${name}_wheel_joint">
+        <hardwareInterface>hardware_interface/VelocityJointInterface</hardwareInterface>
+      </joint>
+    </transmission> -->
+    <!-- <gazebo reference="${name}_wheel_link">
+      <material>Gazebo/Yellow</material>
+    </gazebo> -->
+  </xacro:macro>
+  <!-- Bicycle model front wheel link (passive - no transmission) -->
+  <xacro:macro name="front_wheel"
     params="
       name
@@ -207,52 +257,4 @@
       <axis xyz="0 0 1"/>
     </joint>
-    <!-- <transmission name="${name}_wheel_joint_trans">
-      <type>transmission_interface/SimpleTransmission</type>
-      <actuator name="${name}_wheel_joint_motor">
-        <mechanicalReduction>1</mechanicalReduction>
-        <hardwareInterface>hardware_interface/VelocityJointInterface</hardwareInterface>
-      </actuator>
-      <joint name="${name}_wheel_joint">
-        <hardwareInterface>hardware_interface/VelocityJointInterface</hardwareInterface>
-      </joint>
-    </transmission> -->
-    <gazebo reference="${name}_wheel_link">
-      <material>Gazebo/Yellow</material>
-    </gazebo>
-  </xacro:macro>
-  <!-- Bicycle model front wheel link (passive - no transmission) -->
-  <xacro:macro name="front_wheel"
-    params="
-      name
-      parent
-      wheel_radius
-      wheel_thickness
-      wheel_mass
-      *origin">
-    <link name="${name}_wheel_link">
-      <visual>
-        <origin xyz="0 0 0" rpy="0 0 0"/>
-        <geometry>
-          <cylinder radius="${wheel_radius}" length="${wheel_thickness}"/>
-        </geometry>
-        <material name="yellow" />
-      </visual>
-      <collision>
-        <origin xyz="0 0 0" rpy="0 0 0"/>
-        <geometry>
-          <cylinder radius="${wheel_radius}" length="${wheel_thickness}"/>
-        </geometry>
-      </collision>
-      <xacro:solid_cylinder_inertial
-          rpy="0 0 0" xyz="0 0 0"
-          mass="${wheel_mass}"
-          radius="${wheel_radius}" length="${wheel_thickness}" />
-    </link>
-    <joint name="${name}_wheel_joint" type="continuous">
-      <parent link="${parent}_link"/>
-      <child link="${name}_wheel_link"/>
-      <xacro:insert_block name="origin"/>
-      <axis xyz="0 0 1"/>
-    </joint>
     <gazebo reference="${name}_wheel_link">
       <material>Gazebo/Yellow</material>
@@ -267,14 +269,19 @@
       name
       parent
+      reflect
       wheel_radius
       wheel_thickness
       wheel_mass
-      *origin">
+      base_length
+      base_width
+      axle_offset
+      axle_height">
+      <!-- *origin"> -->
     <link name="${name}_wheel_link">
       <visual>
-        <origin xyz="0 0 0" rpy="0 0 0"/>
-        <geometry>
-          <cylinder radius="${wheel_radius}" length="${wheel_thickness}"/>
-					<!-- <mesh filename="package://robotrendszerek_projekt/meshes/f1_car_wheel.dae"/> -->
+        <origin xyz="0 0 0" rpy="${(1-reflect)/2 * 180 * deg_to_rad} 0 0"/>
+        <geometry>
+          <!-- <cylinder radius="${wheel_radius}" length="${wheel_thickness}"/> -->
+          <mesh filename="package://race_car_gazebo/meshes/f1_car_wheel_rear.dae"/>
         </geometry>
         <material name="red" />
@@ -294,5 +301,7 @@
       <parent link="${parent}_link"/>
       <child link="${name}_wheel_link"/>
-      <xacro:insert_block name="origin"/>
+      <!-- <xacro:insert_block name="origin"/> -->
+      <origin xyz="${-base_length/2+axle_offset_rear} ${reflect * (+base_width/2-wheel_thickness/2)} ${axle_height}"
+              rpy="${-90 * deg_to_rad} 0 0"/>
       <axis xyz="0 0 1"/>
     </joint>
@@ -308,9 +317,9 @@
     </transmission> -->
     <gazebo reference="${name}_wheel_link">
-      <material>Gazebo/Red</material>
+      <!-- <material>Gazebo/Red</material> -->
       <mu1 value="1.0"/>
 			<mu2 value="1.0"/>
-			<kp value="10000000.0" />
-			<kd value="1.0" />
+			<kp value="100000.0" />
+			<kd value="10.0" />
 			<fdir1 value="1 0 0"/>
     </gazebo>
