Commit message: Kamera szenzor hozzáadva

File: race_car_description/urdf/f1_car.xacro (robot description, xacro)
@@ -16,6 +16,7 @@
 -->
 <robot name="f1_car" xmlns:xacro="http://wiki.ros.org/xacro">
-  <!-- Include xacro for inertials, materials and wheels -->
+  <!-- Include xacro for inertials, materials, wheels and camera -->
   <xacro:include filename="$(find race_car_description)/urdf/wheel.xacro"/>
+  <xacro:include filename="$(find race_car_description)/urdf/camera.xacro"/>
   <xacro:property name="robot_namespace" value="/"/>
   <!-- <xacro:property name="robot_namespace" value="/f1_car"/> -->
@@ -33,17 +34,18 @@
   <!-- Math constants -->
   <xacro:property name="deg_to_rad" value="0.01745329251994329577"/>
+  <xacro:property name="mass_multiplier" value="10"/>
   <!-- Robot base dimensions -->
   <xacro:property name="base_length" value="${5.5 / 32}" />
   <xacro:property name="base_width" value="${2.0 / 32}" />
   <xacro:property name="base_height" value="${1.0 / 32}" />
-  <xacro:property name="base_mass" value="0.025" />
+  <xacro:property name="base_mass" value="${0.025 * mass_multiplier}" />
   <!-- Wheel link dimensions -->
   <xacro:property name="wheel_radius" value="${18*0.0254/2 / 32}" />
   <xacro:property name="wheel_thickness" value="${0.35 / 32}" />
-  <xacro:property name="wheel_mass" value="0.00032" />
+  <xacro:property name="wheel_mass" value="${0.00032 * mass_multiplier}" />
   <!-- Steering link dimensions -->
   <xacro:property name="steer_radius" value="${wheel_radius / 2}" />
   <xacro:property name="steer_thickness" value="${wheel_thickness / 4}" />
-  <xacro:property name="steer_mass" value="0.00032" />
+  <xacro:property name="steer_mass" value="${0.00032 * mass_multiplier}" />
   <!-- Axle positions -->
   <xacro:property name="wheelbase" value="${3.6 / 32}" />
@@ -54,4 +56,11 @@
   <xacro:property name="axle_height" value="${-base_height/2 - ride_height + wheel_radius}" />
   <xacro:property name="steer_offset" value="${steer_thickness}" />
+  <!-- Camera dimensions -->
+	<xacro:property name="camera_size" value="${0.2 / 32}"/>
+	<xacro:property name="camera_width" value="${camera_size}"/>
+	<xacro:property name="camera_thickness" value="${camera_size/2}"/>
+	<xacro:property name="camera_height" value="${camera_size*2/3}"/>
+	<xacro:property name="camera_mass" value="${0.00003 * mass_multiplier}"/>
+	<xacro:property name="camera_forward_tilt_deg" value="0"/>
   <!-- Base link -->
   <link name="base_link">
@@ -74,4 +83,14 @@
         x="${base_length}" y="${base_width}" z="${base_height}" />
   </link>
+  <!-- Camera -->
+  <xacro:camera
+    parent="base_link"
+    camera_width="${camera_width}"
+    camera_thickness="${camera_thickness}"
+    camera_height="${camera_height}"
+    forward_tilt="${camera_forward_tilt_deg}">
+    <origin xyz="${base_length/2+camera_thickness/2} 0 ${base_height/2-camera_height/2}"
+            rpy="0 ${camera_forward_tilt_deg * deg_to_rad} 0"/>
+  </xacro:camera>
   <!-- Front steer and rear wheel joints required for ackermann_steering_controller -->
   <xacro:front_steer

File: race_car_description/urdf/inertials.xacro (robot description, xacro)
@@ -8,4 +8,7 @@
  -->
 <robot name="inertials" xmlns:xacro="http://wiki.ros.org/xacro">
+    <xacro:property name="include_guard_inertials" default="true"/>
+    <xacro:if value="${include_guard_inertials}">
+    <xacro:property name="include_guard_inertials" value="false"/>
     <!-- Math constants -->
     <xacro:property name="math_pi"        value="3.141592653589793" />
@@ -41,3 +44,4 @@
         </inertial>
     </xacro:macro>
+    </xacro:if>
 </robot>

File: race_car_description/urdf/materials.xacro (robot description, xacro)
@@ -1,4 +1,7 @@
 <?xml version="1.0"?>
-<robot>
+<robot name="materials" xmlns:xacro="http://wiki.ros.org/xacro">
+  <xacro:property name="include_guard_materials" default="true"/>
+  <xacro:if value="${include_guard_materials}">
+  <xacro:property name="include_guard_materials" value="false"/>
   <material name="black">
     <color rgba="0.0 0.0 0.0 1.0"/>
@@ -34,3 +37,4 @@
     <color rgba="${222/255} ${207/255} ${195/255} 1.0"/>
   </material>
+  </xacro:if>
 </robot>

Commit message: Vonalkövetés megvalósítása

File: race_car_description/urdf/f1_car.xacro (robot description, xacro)
@@ -34,5 +34,5 @@
   <!-- Math constants -->
   <xacro:property name="deg_to_rad" value="0.01745329251994329577"/>
-  <xacro:property name="mass_multiplier" value="10"/>
+  <xacro:property name="mass_multiplier" value="1"/>
   <xacro:property name="scale" value="32"/>
   <!-- Robot base dimensions -->
@@ -67,9 +67,8 @@
 	<!-- <xacro:property name="camera_x" value="${base_length/2+camera_thickness/2}"/> -->
 	<xacro:property name="camera_y" value="0"/>
-	<!-- <xacro:property name="camera_z" value="${base_height/2-camera_height/2}"/> -->
-	<!-- <xacro:property name="camera_x" value="${-1.41 / scale + camera_thickness/2}"/>
-	<xacro:property name="camera_z" value="${0.82 / scale - camera_height/2}"/> -->
-	<xacro:property name="camera_x" value="${2.75 / scale + camera_thickness/2}"/>
-	<xacro:property name="camera_z" value="${-0.192 / scale - camera_height/2}"/>
+	<xacro:property name="camera_x" value="${base_length/2 + camera_thickness/2}"/>
+	<xacro:property name="camera_z" value="${base_height/2-camera_height/2}"/>
+	<!-- <xacro:property name="camera_x" value="${2.75 / scale + camera_thickness/2}"/> -->
+	<!-- <xacro:property name="camera_z" value="${-0.192 / scale - camera_height/2}"/> -->
   <!-- Base link -->
   <link name="base_link">
@@ -123,7 +122,7 @@
     name="rear"
     parent="base"
-    wheel_radius="${wheel_radius/4}"
-    wheel_thickness="${wheel_thickness/2}"
-    wheel_mass="${wheel_mass/32}">
+    wheel_radius="${wheel_radius}"
+    wheel_thickness="${wheel_thickness}"
+    wheel_mass="${wheel_mass}">
     <origin xyz="${-base_length/2+axle_offset_rear} 0 ${axle_height}" rpy="${-90 * deg_to_rad} 0 0"/>
   </xacro:rear_wheel>

File: race_car_description/urdf/wheel.xacro (robot description, xacro)
@@ -168,9 +168,10 @@
     <gazebo reference="${name}_wheel_link">
       <!-- <material>Gazebo/Red</material> -->
-      <mu1 value="1.0"/>
-			<mu2 value="1.0"/>
+      <mu1 value="1.5"/>
+			<mu2 value="1.5"/>
 			<kp value="100000.0" />
 			<kd value="10.0" />
 			<fdir1 value="1 0 0"/>
+      <dampingFactor value="0.70"/>
     </gazebo>
   </xacro:macro>
@@ -318,9 +319,10 @@
     <gazebo reference="${name}_wheel_link">
       <!-- <material>Gazebo/Red</material> -->
-      <mu1 value="1.0"/>
-			<mu2 value="1.0"/>
+      <mu1 value="1.5"/>
+			<mu2 value="1.5"/>
 			<kp value="100000.0" />
 			<kd value="10.0" />
 			<fdir1 value="1 0 0"/>
+      <dampingFactor value="0.70"/>
     </gazebo>
   </xacro:macro>
